File: HappyDay_ATM90e26_Kicad.kicad_pcb (KiCad board)
At the start: 2 copper layers, 103 x 51.5 mm, 86 parts, among them J1 Conn_01x03, J10 GS3, J11 GS3, J17 GS3, J18 GS3, J2 TRS3.5Female, J3 TRS3.5Female, M1 ATM90E26_ATM90E26, M2 ATM90E26_ATM90E26, U1 RAC03-3.3SGA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

Commit message: added image of PCBs got back from OSHPark
Parts:
- C1, C13, C14, C16, C2, C5, L1, R10, R11, R12, R20, R21, R22, R23: moved to B.Cu
- TP1, TP10, TP11, TP2, TP3, TP4, TP6, TP7, TP8, TP9: footprint Connectors_TestPoints:Test_Point_Pad_d2.0mm -> Connectors_TestPoints:Test_Point_Loop_D2.54mm_Drill1.5mm_Beaded
- U3: footprint HappyDayEnergyMonitor:Si865 -> HappyDayEnergyMonitor:SOIC-16
- moved TP2 45.8 mm to (117.2, 69.7)
- moved TP4 27.6 mm to (87.2, 79.9)
- moved TP9 27.4 mm to (77.5, 116.5)
- moved TP7 20.4 mm to (86.2, 105.1)
- moved TP3 17.9 mm to (108.8, 69.8)
- moved TP8 16.2 mm to (88.3, 116.6)
- moved C16 12.7 mm to (95.5, 101.4), turned to 180 degrees
- moved R4 12.4 mm to (75.9, 73.9)
- moved R8 12.3 mm to (87.1, 73.6)
- moved R6 12.0 mm to (81.6, 73.8)
- moved TP6 11.6 mm to (80.5, 105.1)
- moved R12 11.5 mm to (91.7, 77.7)
- moved R19 10.8 mm to (110.3, 112.7), turned to 0 degrees
- moved R3 10.6 mm to (76.0, 69.8)
- moved R5 10.4 mm to (81.5, 69.8)
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Routing:
- net Net-(R19-Pad2): track 22.7 -> 2.93 mm
- net L0: track 62.0 -> 77.6 mm, vias 4 -> 3
- net I1N_0: track 29.7 -> 44.8 mm, vias 3 -> 1
- net CS1_ATM: track 2.65 -> 17.5 mm, vias 1 -> 3
- net N: track 82.0 -> 96.7 mm, vias 8 -> 2
- net L0_SAMP: track 26.4 -> 37.2 mm, vias 2 -> 3
- net Net-(R23-Pad2): track 14.3 -> 3.82 mm, vias 0 -> 1
- net I1P_0: track 46.6 -> 55.1 mm, vias 3 -> 5
- net Net-(C4-Pad2): track 32.0 -> 39.8 mm, vias 0 -> 3
- net L1_SAMP: track 46.7 -> 54.0 mm, vias 0 -> 7
- net MISO_MCU: track 25.8 -> 32.4 mm, vias 0 -> 2
- net Net-(D2-Pad1): track 9.65 -> 3.23 mm
- net Net-(R22-Pad2): track 5.06 -> 9.99 mm, vias 0 -> 1
- net Net-(J3-Pad2): track 18.1 -> 13.3 mm, vias 2 -> 3
- net SCLK_MCU: track 33.8 -> 29.0 mm
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Other:
- board size 103 x 51.5 mm -> 103 x 52.3 mm
