File: HappyDay_ATM90e26_Kicad.sch (KiCad schematic (older format))
At the start: 46 parts, among them J1 Conn_01x03, J2 TRS3.5Female, J3 TRS3.5Female, U1 RAC03-3.3SGA, U2 dc-dc

Commit message: added image of PCBs got back from OSHPark
Parts:
- TP1, TP2, TP3, TP4, TP6, TP7, TP8, TP9: footprint Connectors_TestPoints:Test_Point_Pad_d2.0mm -> Connectors_TestPoints:Test_Point_Loop_D2.54mm_Drill1.5mm_Beaded
Changed lines of the file:
@@
 EESchema Schematic File Version 2
-LIBS:HappyDay_Energy_PCB-rescue
 LIBS:power
 LIBS:device
@@
 LIBS:si865
 LIBS:MiscellaneousDevices
-LIBS:HappyDay_Energy_PCB-cache
+LIBS:HappyDay_ATM90e26_Kicad-cache
 EELAYER 25 0
 EELAYER END
@@
 F 0 "TP1" H 6250 3700 50  0000 C BNN
 F 1 "3.3V_A" H 6250 3650 50  0000 C CNN
-F 2 "Connectors_TestPoints:Test_Point_Pad_d2.0mm" H 6250 3400 50  0001 C CNN
+F 2 "Connectors_TestPoints:Test_Point_Loop_D2.54mm_Drill1.5mm_Beaded" H 6250 3400 50  0001 C CNN
 F 3 "" H 6250 3400 50  0001 C CNN
 F 4 "X" H 6250 3400 60  0001 C CNN "PN"
@@
 F 0 "TP2" H 6250 4150 50  0000 C BNN
 F 1 "GNDA" H 6250 4100 50  0000 C CNN
-F 2 "Connectors_TestPoints:Test_Point_Pad_d2.0mm" H 6250 3850 50  0001 C CNN
+F 2 "Connectors_TestPoints:Test_Point_Loop_D2.54mm_Drill1.5mm_Beaded" H 6250 3850 50  0001 C CNN
 F 3 "" H 6250 3850 50  0001 C CNN
 F 4 "X" H 6250 3850 60  0001 C CNN "PN"
@@
 F 0 "TP3" H 6250 4550 50  0000 C BNN
 F 1 "LO_SAMP" H 6250 4500 50  0000 C CNN
-F 2 "Connectors_TestPoints:Test_Point_Pad_d2.0mm" H 6250 4250 50  0001 C CNN
+F 2 "Connectors_TestPoints:Test_Point_Loop_D2.54mm_Drill1.5mm_Beaded" H 6250 4250 50  0001 C CNN
 F 3 "" H 6250 4250 50  0001 C CNN
 F 4 "X" H 6250 4250 60  0001 C CNN "PN"
@@
 F 0 "TP4" H 6250 4950 50  0000 C BNN
 F 1 "L1_SAMP" H 6250 4900 50  0000 C CNN
-F 2 "Connectors_TestPoints:Test_Point_Pad_d2.0mm" H 6250 4650 50  0001 C CNN
+F 2 "Connectors_TestPoints:Test_Point_Loop_D2.54mm_Drill1.5mm_Beaded" H 6250 4650 50  0001 C CNN
 F 3 "" H 6250 4650 50  0001 C CNN
 F 4 "x" H 6250 4650 60  0001 C CNN "PN"
@@
 F 0 "TP6" H 6250 5750 50  0000 C BNN
 F 1 "I1P_0" H 6250 5700 50  0000 C CNN
-F 2 "Connectors_TestPoints:Test_Point_Pad_d2.0mm" H 6250 5450 50  0001 C CNN
+F 2 "Connectors_TestPoints:Test_Point_Loop_D2.54mm_Drill1.5mm_Beaded" H 6250 5450 50  0001 C CNN
 F 3 "" H 6250 5450 50  0001 C CNN
 F 4 "x" H 6250 5450 60  0001 C CNN "PN"
@@
 F 0 "TP7" H 6250 6150 50  0000 C BNN
 F 1 "I1N_0" H 6250 6100 50  0000 C CNN
-F 2 "Connectors_TestPoints:Test_Point_Pad_d2.0mm" H 6250 5850 50  0001 C CNN
+F 2 "Connectors_TestPoints:Test_Point_Loop_D2.54mm_Drill1.5mm_Beaded" H 6250 5850 50  0001 C CNN
 F 3 "" H 6250 5850 50  0001 C CNN
 F 4 "x" H 6250 5850 60  0001 C CNN "PN"
@@
 F 0 "TP8" H 6250 6550 50  0000 C BNN
 F 1 "I1P_1" H 6250 6500 50  0000 C CNN
-F 2 "Connectors_TestPoints:Test_Point_Pad_d2.0mm" H 6250 6250 50  0001 C CNN
+F 2 "Connectors_TestPoints:Test_Point_Loop_D2.54mm_Drill1.5mm_Beaded" H 6250 6250 50  0001 C CNN
 F 3 "" H 6250 6250 50  0001 C CNN
 F 4 "x" H 6250 6250 60  0001 C CNN "PN"
@@
 F 0 "TP9" H 10550 3800 50  0000 C BNN
 F 1 "I1N_1" H 10550 3750 50  0000 C CNN
-F 2 "Connectors_TestPoints:Test_Point_Pad_d2.0mm" H 10550 3500 50  0001 C CNN
+F 2 "Connectors_TestPoints:Test_Point_Loop_D2.54mm_Drill1.5mm_Beaded" H 10550 3500 50  0001 C CNN
 F 3 "" H 10550 3500 50  0001 C CNN
 F 4 "x" H 10550 3500 60  0001 C CNN "PN"

Commit message: added Schematic_top_sheet.png
Other:
- note added: "120VAC -> +3.3VDC Power Supply\n"
- note added: "2 x 120 VAC In"
- note added: "DC (ATM90E26) - DC (Feather) Isolation"
- note added: "Transformer"
- note removed: "120VAC -> +3.3VDC Regulated\n"
- note removed: "3.3V For ATM isolated from 3.3V for MCU"
- note removed: "Energy In"
Changed lines of the file:
@@
 	1    0    0    -1
 $EndComp
-Text Notes 1250 650  0    60   ~ 0
-Energy In
-Text Notes 3350 650  0    60   ~ 0
+Text Notes 700  800  0    120  ~ 0
+2 x 120 VAC In
+Text Notes 3350 650  0    100  ~ 0
 Sample Voltage\n
 $Comp
@@
 Text GLabel 9800 1750 3    60   Input ~ 0
 3.3V_MCU
-Text Notes 1400 2700 0    60   ~ 0
+Text Notes 1250 2750 0    120  ~ 0
 Sample Current\n
 $Comp
@@
 Text GLabel 8100 1400 2    60   Output ~ 0
 3.3V_MCU
-Text Notes 6400 700  0    60   ~ 0
-120VAC -> +3.3VDC Regulated\n
+Text Notes 5900 750  0    120  ~ 0
+120VAC -> +3.3VDC Power Supply\n
 $Sheet
 S 6500 3200 3750 3250
@@
 F12 "3.3V_MCU" I R 10250 3900 60
 $EndSheet
-Text Notes 7200 3700 0    60   ~ 0
+Text Notes 7500 4450 0    120  ~ 0
 Measure and Send
 $Comp
@@
 Wire Wire Line
 	8100 1900 8100 1850
-Wire Notes Line
-	8850 450  8850 3150
 Wire Wire Line
 	8100 2250 8100 2200
@@
 	1    0    0    -1
 $EndComp
-Text Notes 9000 700  0    60   ~ 0
-3.3V For ATM isolated from 3.3V for MCU
+Text Notes 8850 1000 0    60   ~ 0
+DC (ATM90E26) - DC (Feather) Isolation
+Wire Bus Line
+	3900 5650 3900 2450
+Text Notes 6850 1050 0    60   ~ 0
+Transformer
 $EndSCHEMATC
