File: HappyDay_ATM90e26_Kicad.sch (KiCad schematic (older format))
At the start: 46 parts, among them J1 Conn_01x03, J2 TRS3.5Female, J3 TRS3.5Female, U1 RAC03-3.3SGA, U2 dc-dc

Commit message: Version b (#1)
* added readme.md to version_B

* added image of PCBs got back from OSHPark

* added image of PCBs got back from OSHPark

* added image of PCBs got back from OSHPark

* added kicad image of voltage sampling

* added voltage sampling test setup image

* added danger electricity image

* updated danger electricity image

* added current sampling kicad image

* added Arduino_AC_current_input_A.png image from OEM site

* added TRS_connector.png

* added scope_current_IP0_andIP1.png

* added test_lamp.jpg

* added RAC03-3.3SGA.png

* added cme0303s3c.png

* modified cme0303S3c.png

* added atm90e26_soldered_on_pcb.jpg

* added atm90e26_schematic.png;

* added Feather_on_PCB.jpg

* add Feather_pins_Schematic.png

* added Schematic_top_sheet.png

* added sense_power_cable.png

* added front_PCB_itemized.png

* added back_PCB_itemized.png

* added Schematic_meter_sheet.png

* added RAC03-caps-from-datasheet.png

* added atm90e26_short_circuit_solder.png

* added PCB_Layout_first_atm90e26_pins.png

* added Logic_analyzer_error.png
Parts:
- TP1, TP2, TP3, TP4, TP6, TP7, TP8, TP9: footprint Connectors_TestPoints:Test_Point_Pad_d2.0mm -> Connectors_TestPoints:Test_Point_Loop_D2.54mm_Drill1.5mm_Beaded
Other:
- note added: "120VAC -> +3.3VDC Power Supply\n"
- note added: "2 x 120 VAC In"
- note added: "DC (ATM90E26) - DC (Feather) Isolation"
- note added: "Transformer"
- note removed: "120VAC -> +3.3VDC Regulated\n"
- note removed: "3.3V For ATM isolated from 3.3V for MCU"
- note removed: "Energy In"
Changed lines of the file:
@@
 EESchema Schematic File Version 2
-LIBS:HappyDay_Energy_PCB-rescue
 LIBS:power
 LIBS:device
@@
 LIBS:si865
 LIBS:MiscellaneousDevices
-LIBS:HappyDay_Energy_PCB-cache
+LIBS:HappyDay_ATM90e26_Kicad-cache
 EELAYER 25 0
 EELAYER END
@@
 	1    0    0    -1
 $EndComp
-Text Notes 1250 650  0    60   ~ 0
-Energy In
-Text Notes 3350 650  0    60   ~ 0
+Text Notes 700  800  0    120  ~ 0
+2 x 120 VAC In
+Text Notes 3350 650  0    100  ~ 0
 Sample Voltage\n
 $Comp
@@
 Text GLabel 9800 1750 3    60   Input ~ 0
 3.3V_MCU
-Text Notes 1400 2700 0    60   ~ 0
+Text Notes 1250 2750 0    120  ~ 0
 Sample Current\n
 $Comp
@@
 Text GLabel 8100 1400 2    60   Output ~ 0
 3.3V_MCU
-Text Notes 6400 700  0    60   ~ 0
-120VAC -> +3.3VDC Regulated\n
+Text Notes 5900 750  0    120  ~ 0
+120VAC -> +3.3VDC Power Supply\n
 $Sheet
 S 6500 3200 3750 3250
@@
 F12 "3.3V_MCU" I R 10250 3900 60
 $EndSheet
-Text Notes 7200 3700 0    60   ~ 0
+Text Notes 7500 4450 0    120  ~ 0
 Measure and Send
 $Comp
@@
 Wire Wire Line
 	8100 1900 8100 1850
-Wire Notes Line
-	8850 450  8850 3150
 Wire Wire Line
 	8100 2250 8100 2200
@@
 F 0 "TP1" H 6250 3700 50  0000 C BNN
 F 1 "3.3V_A" H 6250 3650 50  0000 C CNN
-F 2 "Connectors_TestPoints:Test_Point_Pad_d2.0mm" H 6250 3400 50  0001 C CNN
+F 2 "Connectors_TestPoints:Test_Point_Loop_D2.54mm_Drill1.5mm_Beaded" H 6250 3400 50  0001 C CNN
 F 3 "" H 6250 3400 50  0001 C CNN
 F 4 "X" H 6250 3400 60  0001 C CNN "PN"
@@
 F 0 "TP2" H 6250 4150 50  0000 C BNN
 F 1 "GNDA" H 6250 4100 50  0000 C CNN
-F 2 "Connectors_TestPoints:Test_Point_Pad_d2.0mm" H 6250 3850 50  0001 C CNN
+F 2 "Connectors_TestPoints:Test_Point_Loop_D2.54mm_Drill1.5mm_Beaded" H 6250 3850 50  0001 C CNN
 F 3 "" H 6250 3850 50  0001 C CNN
 F 4 "X" H 6250 3850 60  0001 C CNN "PN"
@@
 F 0 "TP3" H 6250 4550 50  0000 C BNN
 F 1 "LO_SAMP" H 6250 4500 50  0000 C CNN
-F 2 "Connectors_TestPoints:Test_Point_Pad_d2.0mm" H 6250 4250 50  0001 C CNN
+F 2 "Connectors_TestPoints:Test_Point_Loop_D2.54mm_Drill1.5mm_Beaded" H 6250 4250 50  0001 C CNN
 F 3 "" H 6250 4250 50  0001 C CNN
 F 4 "X" H 6250 4250 60  0001 C CNN "PN"
@@
 F 0 "TP4" H 6250 4950 50  0000 C BNN
 F 1 "L1_SAMP" H 6250 4900 50  0000 C CNN
-F 2 "Connectors_TestPoints:Test_Point_Pad_d2.0mm" H 6250 4650 50  0001 C CNN
+F 2 "Connectors_TestPoints:Test_Point_Loop_D2.54mm_Drill1.5mm_Beaded" H 6250 4650 50  0001 C CNN
 F 3 "" H 6250 4650 50  0001 C CNN
 F 4 "x" H 6250 4650 60  0001 C CNN "PN"
@@
 F 0 "TP6" H 6250 5750 50  0000 C BNN
 F 1 "I1P_0" H 6250 5700 50  0000 C CNN
-F 2 "Connectors_TestPoints:Test_Point_Pad_d2.0mm" H 6250 5450 50  0001 C CNN
+F 2 "Connectors_TestPoints:Test_Point_Loop_D2.54mm_Drill1.5mm_Beaded" H 6250 5450 50  0001 C CNN
 F 3 "" H 6250 5450 50  0001 C CNN
 F 4 "x" H 6250 5450 60  0001 C CNN "PN"
@@
 F 0 "TP7" H 6250 6150 50  0000 C BNN
 F 1 "I1N_0" H 6250 6100 50  0000 C CNN
-F 2 "Connectors_TestPoints:Test_Point_Pad_d2.0mm" H 6250 5850 50  0001 C CNN
+F 2 "Connectors_TestPoints:Test_Point_Loop_D2.54mm_Drill1.5mm_Beaded" H 6250 5850 50  0001 C CNN
 F 3 "" H 6250 5850 50  0001 C CNN
 F 4 "x" H 6250 5850 60  0001 C CNN "PN"
@@
 F 0 "TP8" H 6250 6550 50  0000 C BNN
 F 1 "I1P_1" H 6250 6500 50  0000 C CNN
-F 2 "Connectors_TestPoints:Test_Point_Pad_d2.0mm" H 6250 6250 50  0001 C CNN
+F 2 "Connectors_TestPoints:Test_Point_Loop_D2.54mm_Drill1.5mm_Beaded" H 6250 6250 50  0001 C CNN
 F 3 "" H 6250 6250 50  0001 C CNN
 F 4 "x" H 6250 6250 60  0001 C CNN "PN"
@@
 F 0 "TP9" H 10550 3800 50  0000 C BNN
 F 1 "I1N_1" H 10550 3750 50  0000 C CNN
-F 2 "Connectors_TestPoints:Test_Point_Pad_d2.0mm" H 10550 3500 50  0001 C CNN
+F 2 "Connectors_TestPoints:Test_Point_Loop_D2.54mm_Drill1.5mm_Beaded" H 10550 3500 50  0001 C CNN
 F 3 "" H 10550 3500 50  0001 C CNN
 F 4 "x" H 10550 3500 60  0001 C CNN "PN"
@@
 	1    0    0    -1
 $EndComp
-Text Notes 9000 700  0    60   ~ 0
-3.3V For ATM isolated from 3.3V for MCU
+Text Notes 8850 1000 0    60   ~ 0
+DC (ATM90E26) - DC (Feather) Isolation
+Wire Bus Line
+	3900 5650 3900 2450
+Text Notes 6850 1050 0    60   ~ 0
+Transformer
 $EndSCHEMATC

Commit message: modified current_sampling_Kicad.png
Parts:
- removed TP1: 3.3V_A, Connectors_TestPoints:Test_Point_Loop_D2.54mm_Drill1.5mm_Beaded, symbol TEST
- removed TP10: 3.3V_D, Connectors_TestPoints:Test_Point_Pad_d2.0mm, symbol TEST
- removed TP11: GND_D, Connectors_TestPoints:Test_Point_Pad_d2.0mm, symbol TEST
- removed TP2: GNDA, Connectors_TestPoints:Test_Point_Loop_D2.54mm_Drill1.5mm_Beaded, symbol TEST
- removed U2: dc-dc, HappyDayEnergyMonitor:DC-DC, symbol dc-dc
- added L2: Ferrite SM, Capacitors_SMD:C_0805, symbol L_Core_Ferrite_Small
Connections:
- net labels added: GNDD, IN_0, IN_1, IP_0, IP_1, LO, LO_SAMP
- net labels removed: 3.3V_MCU, 3.3V_REG_A, GND_MCU, I1N_0, I1N_1, I1P_0, I1P_1, L0, L0_SAMP
- wire segments 96 -> 87
Other:
- note removed: "DC (ATM90E26) - DC (Feather) Isolation"

Commit message: updated design and layout sent to OSH Park (2/26/2018)
Parts:
- removed J2, J3: TRS3.5Female, HappyDayEnergyMonitor:Audio-Jack, symbol TRS3.5Female
- removed L2: Ferrite SM, Capacitors_SMD:C_0805, symbol L_Core_Ferrite_Small
- added J2, J3: TRS3.5, HappyDayEnergyMonitor:Audio-Jack, symbol TRS3.5
- added TP1: GNDD, Connectors_TestPoints:Test_Point_Loop_D2.54mm_Drill1.5mm_Beaded, symbol TEST
- added TP2: 3.3V, Connectors_TestPoints:Test_Point_Loop_D2.54mm_Drill1.5mm_Beaded, symbol TEST
- added TP5: GNDA, Connectors_TestPoints:Test_Point_Loop_D2.54mm_Drill1.5mm_Beaded, symbol TEST
- F1: PN LVR005NK -> 0ZRE0012FF1C
- L1: PN HI1206T500R-10 -> AIML-1206-R27K-T
- TP6: value I1P_0 -> IP_0
- TP7: value I1N_0 -> IN_0
- TP8: value I1P_1 -> IP_1
- TP9: value I1N_1 -> IN_1
Connections:
- wire segments 87 -> 89
Changed lines of the file:
@@
 F 2 "Capacitors_SMD:C_1206" V 1330 1650 50  0001 C CNN
 F 3 "" H 1400 1650 50  0001 C CNN
-F 4 "HI1206T500R-10" H 1400 1650 60  0001 C CNN "PN"
+F 4 "AIML-1206-R27K-T" H 1400 1650 60  0001 C CNN "PN"
 	1    1400 1650
 	1    0    0    -1
@@
 F 2 "HappyDayEnergyMonitor:POLYFUSE" H 7750 1900 50  0001 L CNN
 F 3 "" H 7700 2100 50  0001 C CNN
-F 4 "LVR005NK" H 7700 2100 60  0001 C CNN "PN"
+F 4 "0ZRE0012FF1C" H 7700 2100 60  0001 C CNN "PN"
 	1    7700 2100
 	0    1    1    0
@@
 F0 "ATM90_Circuit" 60
 F1 "ATM90_Circuit.sch" 60
-F2 "I1P_0" I L 6500 4700 60
-F3 "I1N_0" I L 6500 5150 60
-F4 "L0_SAMP" I L 6500 3500 60
-F5 "N" I L 6500 4300 60
-F6 "I1P_1" I L 6500 5550 60
-F7 "I1N_1" I L 6500 6050 60
-F8 "L1_SAMP" I L 6500 3900 60
+F2 "L0_SAMP" I L 6500 6150 60
+F3 "L1_SAMP" I L 6500 5750 60
+F4 "IP_0" I L 6500 4950 60
+F5 "IN_0" I L 6500 4500 60
+F6 "IP_1" I L 6500 4100 60
+F7 "IN_1" I L 6500 3600 60
 $EndSheet
 Text Notes 7500 4450 0    120  ~ 0
@@
 	0    1    1    0
 $EndComp
-$Comp
-L TRS3.5Female J2
-U 1 1 5A2057E2
-P 1150 3300
-F 0 "J2" H 800 3600 50  0000 C CNN
-F 1 "TRS3.5Female" H 1000 3050 50  0000 C CNN
-F 2 "HappyDayEnergyMonitor:Audio-Jack" H 1400 3400 50  0001 C CNN
-F 3 "" H 1400 3400 50  0001 C CNN
-F 4 "SJ-3523-SMT-TR" H 1150 3300 60  0001 C CNN "PN"
-	1    1150 3300
-	1    0    0    -1
-$EndComp
 Wire Wire Line
 	1450 4000 1450 3450
@@
 Wire Wire Line
 	2050 5400 1450 5400
-$Comp
-L TRS3.5Female J3
-U 1 1 5A205D36
-P 1150 4700
-F 0 "J3" H 800 5000 50  0000 C CNN
-F 1 "TRS3.5Female" H 1000 4450 50  0000 C CNN
-F 2 "HappyDayEnergyMonitor:Audio-Jack" H 1400 4800 50  0001 C CNN
-F 3 "" H 1400 4800 50  0001 C CNN
-F 4 "SJ-3523-SMT-TR" H 1150 4700 60  0001 C CNN "PN"
-	1    1150 4700
-	1    0    0    -1
-$EndComp
 Wire Wire Line
 	1450 5400 1450 4850
@@
 P 6250 4700
 F 0 "TP6" H 6250 5000 50  0000 C BNN
-F 1 "I1P_0" H 6250 4950 50  0000 C CNN
+F 1 "IP_0" H 6250 4950 50  0000 C CNN
 F 2 "Connectors_TestPoints:Test_Point_Loop_D2.54mm_Drill1.5mm_Beaded" H 6250 4700 50  0001 C CNN
 F 3 "" H 6250 4700 50  0001 C CNN
@@
 P 6250 5150
 F 0 "TP7" H 6250 5450 50  0000 C BNN
-F 1 "I1N_0" H 6250 5400 50  0000 C CNN
+F 1 "IN_0" H 6250 5400 50  0000 C CNN
 F 2 "Connectors_TestPoints:Test_Point_Loop_D2.54mm_Drill1.5mm_Beaded" H 6250 5150 50  0001 C CNN
 F 3 "" H 6250 5150 50  0001 C CNN
@@
 P 6250 5550
 F 0 "TP8" H 6250 5850 50  0000 C BNN
-F 1 "I1P_1" H 6250 5800 50  0000 C CNN
+F 1 "IP_1" H 6250 5800 50  0000 C CNN
 F 2 "Connectors_TestPoints:Test_Point_Loop_D2.54mm_Drill1.5mm_Beaded" H 6250 5550 50  0001 C CNN
 F 3 "" H 6250 5550 50  0001 C CNN
@@
 L TEST TP9
 U 1 1 5A22F1E1
-P 6250 6050
-F 0 "TP9" H 6250 6350 50  0000 C BNN
-F 1 "I1N_1" H 6250 6300 50  0000 C CNN
-F 2 "Connectors_TestPoints:Test_Point_Loop_D2.54mm_Drill1.5mm_Beaded" H 6250 6050 50  0001 C CNN
-F 3 "" H 6250 6050 50  0001 C CNN
-F 4 "x" H 6250 6050 60  0001 C CNN "PN"
-	1    6250 6050
+P 6250 6000
+F 0 "TP9" H 6250 6300 50  0000 C BNN
+F 1 "IN_1" H 6250 6250 50  0000 C CNN
+F 2 "Connectors_TestPoints:Test_Point_Loop_D2.54mm_Drill1.5mm_Beaded" H 6250 6000 50  0001 C CNN
+F 3 "" H 6250 6000 50  0001 C CNN
+F 4 "x" H 6250 6000 60  0001 C CNN "PN"
+	1    6250 6000
 	1    0    0    -1
 $EndComp
@@
 	1    0    0    -1
 $EndComp
-Wire Wire Line
-	4700 1350 4700 1300
 Text Label 5000 800  0    60   ~ 0
 LO_SAMP
@@
 Text Label 7450 2100 0    60   ~ 0
 N
-$Comp
-L L_Core_Ferrite_Small L2
-U 1 1 5A91EC17
-P 9650 1550
-F 0 "L2" H 9700 1590 50  0000 L CNN
-F 1 "Ferrite SM" H 9700 1500 50  0000 L CNN
-F 2 "Capacitors_SMD:C_0805" H 9650 1550 50  0001 C CNN
-F 3 "" H 9650 1550 50  0001 C CNN
-F 4 "MH2029-601Y" H 9650 1550 60  0001 C CNN "PN"
-	1    9650 1550
-	0    1    1    0
-$EndComp
-Wire Wire Line
-	9500 1550 9550 1550
-Wire Wire Line
-	9750 1550 9850 1550
-Wire Wire Line
-	6050 4300 6500 4300
-Text Label 6050 4300 2    60   ~ 0
-N
+Wire Wire Line
+	9500 1550 9850 1550
+Text Label 3050 3900 0    60   ~ 0
+IN_0
 Text Label 3050 3100 0    60   ~ 0
-IN_0
-Text Label 3050 3900 0    60   ~ 0
 IP_0
 Text Label 5950 4700 2    60   ~ 0
@@
 Text Label 5950 5150 2    60   ~ 0
 IN_0
+Text Label 3100 4450 0    60   ~ 0
+IP_1
 Text Label 3100 5250 0    60   ~ 0
-IP_1
-Text Label 3100 4450 0    60   ~ 0
 IN_1
 Text Label 6050 5550 2    60   ~ 0
@@
 Wire Wire Line
 	6500 6050 6050 6050
+$Comp
+L TRS3.5 J2
+U 1 1 5A92CE47
+P 1150 3200
+F 0 "J2" H 800 3500 50  0000 C CNN
+F 1 "TRS3.5" H 1000 2950 50  0000 C CNN
+F 2 "HappyDayEnergyMonitor:Audio-Jack" H 1400 3300 50  0001 C CNN
+F 3 "" H 1400 3300 50  0001 C CNN
+	1    1150 3200
+	1    0    0    1
+$EndComp
+$Comp
+L TRS3.5 J3
+U 1 1 5A92D007
+P 1150 4600
+F 0 "J3" H 800 4900 50  0000 C CNN
+F 1 "TRS3.5" H 1000 4350 50  0000 C CNN
+F 2 "HappyDayEnergyMonitor:Audio-Jack" H 1400 4700 50  0001 C CNN
+F 3 "" H 1400 4700 50  0001 C CNN
+	1    1150 4600
+	1    0    0    1
+$EndComp
+$Comp
+L TEST TP2
+U 1 1 5A93110F
+P 9950 1350
+F 0 "TP2" H 9950 1650 50  0000 C BNN
+F 1 "3.3V" H 9950 1600 50  0000 C CNN
+F 2 "Connectors_TestPoints:Test_Point_Loop_D2.54mm_Drill1.5mm_Beaded" H 9950 1350 50  0001 C CNN
+F 3 "" H 9950 1350 50  0001 C CNN
+F 4 "X" H 9950 1350 60  0001 C CNN "PN"
+	1    9950 1350
+	0    1    1    0
+$EndComp
+$Comp
+L TEST TP1
+U 1 1 5A931745
+P 9950 2400
+F 0 "TP1" H 9950 2700 50  0000 C BNN
+F 1 "GNDD" H 9950 2650 50  0000 C CNN
+F 2 "Connectors_TestPoints:Test_Point_Loop_D2.54mm_Drill1.5mm_Beaded" H 9950 2400 50  0001 C CNN
+F 3 "" H 9950 2400 50  0001 C CNN
+F 4 "X" H 9950 2400 60  0001 C CNN "PN"
+	1    9950 2400
+	0    1    1    0
+$EndComp
+Wire Wire Line
+	9950 2400 9750 2400
+Connection ~ 9750 2400
+Wire Wire Line
+	6250 6000 6250 6050
+Connection ~ 6250 6050
+Wire Wire Line
+	4700 1350 4700 1300
+Connection ~ 4700 1300
+$Comp
+L TEST TP5
+U 1 1 5A944A61
+P 8250 2550
+F 0 "TP5" H 8250 2850 50  0000 C BNN
+F 1 "GNDA" H 8250 2800 50  0000 C CNN
+F 2 "Connectors_TestPoints:Test_Point_Loop_D2.54mm_Drill1.5mm_Beaded" H 8250 2550 50  0001 C CNN
+F 3 "" H 8250 2550 50  0001 C CNN
+F 4 "X" H 8250 2550 60  0001 C CNN "PN"
+	1    8250 2550
+	0    1    1    0
+$EndComp
+Wire Wire Line
+	8250 2550 8100 2550
+Connection ~ 8100 2550
+Wire Wire Line
+	9950 1350 9850 1350
+Connection ~ 9850 1350
 $EndSCHEMATC

Commit message: added eeschema bom xml file
Parts:
- C4: PN (none) -> C; Reference C4 -> (none)
- J2, J3: PN (none) -> SJ-3523-SMT-TR
- U1: PN RAC04-3.3SGB -> RAC03-3.3SGA
Changed lines of the file:
@@
 F 2 "Capacitors_SMD:C_0805" H 8038 1750 50  0001 C CNN
 F 3 "" H 8000 1900 50  0001 C CNN
-F 4 "C4" H 8025 2000 50  0000 L CNN "Reference"
+F 4 "C" H 8000 1900 60  0001 C CNN "PN"
 	1    8000 1900
 	1    0    0    -1
@@
 F 2 "HappyDayEnergyMonitor:RAC03-GA" H 8500 1500 60  0001 C CNN
 F 3 "" H 8500 1500 60  0001 C CNN
-F 4 "RAC04-3.3SGB" H 8900 1750 60  0001 C CNN "PN"
+F 4 "RAC03-3.3SGA" H 8900 1750 60  0001 C CNN "PN"
 	1    8900 1750
 	1    0    0    -1
@@
 F 2 "HappyDayEnergyMonitor:Audio-Jack" H 1400 3300 50  0001 C CNN
 F 3 "" H 1400 3300 50  0001 C CNN
+F 4 "SJ-3523-SMT-TR" H 1150 3200 60  0001 C CNN "PN"
 	1    1150 3200
 	1    0    0    1
@@
 F 2 "HappyDayEnergyMonitor:Audio-Jack" H 1400 4700 50  0001 C CNN
 F 3 "" H 1400 4700 50  0001 C CNN
+F 4 "SJ-3523-SMT-TR" H 1150 4600 60  0001 C CNN "PN"
 	1    1150 4600
 	1    0    0    1
