File: ATM90_Circuit.sch (KiCad schematic (older format))
At the start: 40 parts, among them J10 GS3, J11 GS3, J17 GS3, J18 GS3, M1 ATM90E26_ATM90E26, M2 ATM90E26_ATM90E26, U3 Si865, U4 FeatherHuzzah, Y1 Crystal_Small, Y2 Crystal_Small

Commit message: modified current_sampling_Kicad.png
Parts:
- removed C6, C7: .1u, Capacitors_SMD:C_0805, symbol C
- removed L2, L3: L_Core_Ferrite_Small, Capacitors_SMD:C_0805, symbol L_Core_Ferrite_Small
- removed R14, R15, R16, R17, R18, R19, R20, R21, R22, R23: 51, Capacitors_SMD:C_0805, symbol R
- removed U3: Si865, HappyDayEnergyMonitor:Si865, symbol Si8655
Connections:
- net labels added: IN_0, IP_0
- net labels removed: 3.3V_AVDD, CS0, CS1, GNDA, I1N_0, I1P_0, MISO, MOSI, SCK
- wire segments 188 -> 142
Other:
- note removed: "ATM90e26 Power"

Commit message: modified voltage_sample_voltage_divider.png
Connections:
- net labels added: CS0, MISO, MOSI, SCLK
- net labels removed: CS0_ATM
Changed lines of the file:
@@
 Text HLabel 3950 5800 2    60   Input ~ 0
 N
-Text GLabel 3500 4900 2    60   Input ~ 0
-CS0_ATM
-Text GLabel 3500 4600 2    60   Input ~ 0
-MOSI_ATM
-Text GLabel 3500 4700 2    60   Output ~ 0
-MISO_ATM
-Text GLabel 3500 4800 2    60   Input ~ 0
-SCLK_ATM
 $Comp
 L GS3 J17
@@
 	2100 4600 1800 4600
 Wire Wire Line
-	1800 4150 1800 4600
-Wire Wire Line
-	1350 4150 1800 4150
+	1800 4600 1800 4150
+Wire Wire Line
+	1800 4150 1350 4150
 Wire Wire Line
 	1350 4150 1350 4200
@@
 	6150 4750 5850 4750
 Wire Wire Line
-	5850 4300 5850 4750
-Wire Wire Line
-	5400 4300 5850 4300
+	5850 4750 5850 4300
+Wire Wire Line
+	5850 4300 5400 4300
 Wire Wire Line
 	5400 4300 5400 4350
@@
 Text Label 3500 5000 0    60   ~ 0
 CLKOUT_0
+Text Label 3500 4600 0    60   ~ 0
+MOSI
+Text Label 3500 4700 0    60   ~ 0
+MISO
+Text Label 3500 4800 0    60   ~ 0
+SCLK
+Text Label 3500 4900 0    60   ~ 0
+CS0
 $EndSCHEMATC

Commit message: updated design and layout sent to OSH Park (2/26/2018)
Parts:
- C13, C14, C15, C16: value 27p -> 20p; PN C -> CL21C200JBANNNC
- Y1, Y2: PN ABLS2-3.579545MHZ-D4Y-T -> ABLS3-8.192MHZ-D4Y-T
Connections:
- net labels added: CS1, GNDA, IN_1, IP_1
- net labels removed: +3.3VA, 3.3V_MCU, CS0_MCU, CS1_ATM, CS1_MCU, GNDREF, GND_MCU, I1N_1, I1P_1, MISO_ATM, MISO_MCU, MOSI_ATM, MOSI_MCU, N, SCLK_ATM, SCLK_MCU
- wire segments 142 -> 144

Commit message: changed oscillator caps to 27pf
Parts:
- C13, C14, C15, C16: value 20p -> 27p
Changed lines of the file:
@@
 AR Path="/5A10B9B0" Ref="C13"  Part="1"
 F 0 "C13" H 2525 2850 50  0000 L CNN
-F 1 "20p" H 2525 2650 50  0000 L CNN
+F 1 "27p" H 2525 2650 50  0000 L CNN
 F 2 "Capacitors_SMD:C_0805" H 2538 2600 50  0001 C CNN
 F 3 "" H 2500 2750 50  0001 C CNN
@@
 P 2850 2750
 F 0 "C14" H 2875 2850 50  0000 L CNN
-F 1 "20p" H 2875 2650 50  0000 L CNN
+F 1 "27p" H 2875 2650 50  0000 L CNN
 F 2 "Capacitors_SMD:C_0805" H 2888 2600 50  0001 C CNN
 F 3 "" H 2850 2750 50  0001 C CNN
@@
 P 6450 2900
 F 0 "C15" H 6475 3000 50  0000 L CNN
-F 1 "20p" H 6475 2800 50  0000 L CNN
+F 1 "27p" H 6475 2800 50  0000 L CNN
 F 2 "Capacitors_SMD:C_0805" H 6488 2750 50  0001 C CNN
 F 3 "" H 6450 2900 50  0001 C CNN
@@
 P 6800 2900
 F 0 "C16" H 6825 3000 50  0000 L CNN
-F 1 "20p" H 6825 2800 50  0000 L CNN
+F 1 "27p" H 6825 2800 50  0000 L CNN
 F 2 "Capacitors_SMD:C_0805" H 6838 2750 50  0001 C CNN
 F 3 "" H 6800 2900 50  0001 C CNN

Commit message: added datasheets
Parts:
- removed R24: 10K, Capacitors_SMD:C_0805, symbol R
Connections:
- wire segments 144 -> 142
Changed lines of the file:
@@
 	1    0    0    -1
-$EndComp
-$Comp
-L R R24
-U 1 1 5A20A670
-P 9550 3350
-F 0 "R24" V 9630 3350 50  0000 C CNN
-F 1 "10K" V 9550 3350 50  0000 C CNN
-F 2 "Capacitors_SMD:C_0805" V 9480 3350 50  0001 C CNN
-F 3 "" H 9550 3350 50  0001 C CNN
-F 4 "R" H 9550 3350 60  0001 C CNN "PN"
-	1    9550 3350
-	-1   0    0    1
 $EndComp
 Wire Wire Line
@@
 	9150 4700 9150 4500
 Wire Wire Line
-	9550 3050 9550 3200
-Wire Wire Line
 	8350 3600 9450 3600
-Wire Wire Line
-	9550 3600 9550 3500
 $Comp
 L FeatherHuzzah U4
@@
 Text Label 10050 3450 1    60   ~ 0
 CS0
-$Comp
-L +3.3V #PWR030
-U 1 1 5A92DC7C
-P 9550 3050
-F 0 "#PWR030" H 9550 2900 50  0001 C CNN
-F 1 "+3.3V" H 9550 3190 50  0000 C CNN
-F 2 "" H 9550 3050 50  0001 C CNN
-F 3 "" H 9550 3050 50  0001 C CNN
-	1    9550 3050
-	1    0    0    -1
-$EndComp
 Wire Wire Line
 	7250 4850 7550 4850
